File: hotdog-hw/hotdog-pcb/hotdog-pcb.kicad_sch (KiCad schematic)
At the start: 20 parts, among them J1 Conn_01x01, J2 Conn_01x01, J3 Conn_01x01, J4 Conn_01x01, SW1 SW_SPST, U1 NRF24L01_Breakout, U2 ME2108A

Commit message: Simplify PCB
Parts:
- R6: footprint (none) -> Resistor_THT:R_Axial_DIN0204_L3.6mm_D1.6mm_P5.08mm_Horizontal
- SW1: footprint Button_Switch_THT:SW_Tactile_SPST_Angled_PTS645Vx58-2LFS -> (none)
Connections:
- net at A1.29 (GND), C2.2, R1.2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: now also J3.1 (Pin_1)
- net at A1.4 (GND), C1.2, U1.1 (GND): no longer J3.1 (Pin_1)
Other:
- moved on the sheet: J3
Changed lines of the file:
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@@
   (junction (at 111.76 127) (diameter 0) (color 0 0 0 0)
   )
+  (junction (at 86.36 96.52) (diameter 0) (color 0 0 0 0)
+  )
   (junction (at 137.16 127) (diameter 0) (color 0 0 0 0)
   )
@@
   (junction (at 137.16 96.52) (diameter 0) (color 0 0 0 0)
   )
-  (junction (at 83.82 96.52) (diameter 0) (color 0 0 0 0)
-  )
   (wire (pts (xy 149.86 96.52) (xy 162.56 96.52))
     (stroke (width 0) (type default) (color 0 0 0 0))
@@
   )
   (wire (pts (xy 68.58 81.28) (xy 68.58 71.12))
-    (stroke (width 0) (type default) (color 0 0 0 0))
-  )
-  (wire (pts (xy 83.82 97.79) (xy 83.82 96.52))
     (stroke (width 0) (type default) (color 0 0 0 0))
   )
@@
     (property "Reference" "SW1" (id 0) (at 129.54 30.48 0))
     (property "Value" "SW_SPST" (id 1) (at 129.54 33.02 0))
-    (property "Footprint" "Button_Switch_THT:SW_Tactile_SPST_Angled_PTS645Vx58-2LFS" (id 2) (at 129.54 35.56 0)
+    (property "Footprint" "" (id 2) (at 129.54 35.56 0)
       (effects (font (size 1.27 1.27)) hide)
     )
@@
     (pin "1")
   )
-  (symbol (lib_id "Connector_Generic:Conn_01x01") (at 83.82 102.87 270) (unit 1)
-    (in_bom yes) (on_board yes) (fields_autoplaced)
-    (property "Reference" "J3" (id 0) (at 86.36 101.5999 90)
-      (effects (font (size 1.27 1.27)) (justify left))
-    )
-    (property "Value" "Conn_01x01" (id 1) (at 86.36 104.1399 90)
-      (effects (font (size 1.27 1.27)) (justify left))
-    )
-    (property "Footprint" "Connector_Wire:SolderWire-0.1sqmm_1x01_D0.4mm_OD1mm" (id 2) (at 83.82 102.87 0)
-      (effects (font (size 1.27 1.27)) hide)
-    )
-    (property "Datasheet" "~" (id 3) (at 83.82 102.87 0)
+  (symbol (lib_id "Connector_Generic:Conn_01x01") (at 86.36 101.6 270) (unit 1)
+    (in_bom yes) (on_board yes) (fields_autoplaced)
+    (property "Reference" "J3" (id 0) (at 88.9 100.3299 90)
+      (effects (font (size 1.27 1.27)) (justify left))
+    )
+    (property "Value" "Conn_01x01" (id 1) (at 88.9 102.8699 90)
+      (effects (font (size 1.27 1.27)) (justify left))
+    )
+    (property "Footprint" "Connector_Wire:SolderWire-0.1sqmm_1x01_D0.4mm_OD1mm" (id 2) (at 86.36 101.6 0)
+      (effects (font (size 1.27 1.27)) hide)
+    )
+    (property "Datasheet" "~" (id 3) (at 86.36 101.6 0)
       (effects (font (size 1.27 1.27)) hide)
     )
@@
     (property "Reference" "R6" (id 0) (at 97.79 120.65 90))
     (property "Value" "R" (id 1) (at 97.79 123.19 90))
-    (property "Footprint" "" (id 2) (at 97.79 125.222 90)
+    (property "Footprint" "Resistor_THT:R_Axial_DIN0204_L3.6mm_D1.6mm_P5.08mm_Horizontal" (id 2) (at 97.79 125.222 90)
       (effects (font (size 1.27 1.27)) hide)
     )
@@
     )
     (path "/2d56065f-684a-4165-b0e1-ca322bbb3f18"
-      (reference "SW1") (unit 1) (value "SW_SPST") (footprint "Button_Switch_THT:SW_Tactile_SPST_Angled_PTS645Vx58-2LFS")
+      (reference "SW1") (unit 1) (value "SW_SPST") (footprint "Button_Switch_THT:SW_CuK_OS102011MA1QN1_SPDT_Angled")
     )
     (path "/486e5183-e5a3-4539-8472-387817228f42"
