File: hotdog-hw/hotdog-pcb/hotdog-pcb-front.kicad_pcb (KiCad board)
At the start: 2 copper layers, 202.5 x 50 mm, 29 parts, among them J1 Conn_01x01, J2 Conn_01x01, J3 Conn_01x01, J4 Conn_01x01, SW1 SW_SPST, U1 NRF24L01_Breakout, U2 ME2108A

Commit message: Learned my lesson about PCB pooling
Parts:
- removed D1, D2, D3: LED, LED_THT:LED_D5.0mm
- removed J1, J2: Conn_01x01, Connector_Wire:SolderWire-0.1sqmm_1x01_D0.4mm_OD1mm
- removed R6: R, Resistor_THT:R_Axial_DIN0204_L3.6mm_D1.6mm_P5.08mm_Horizontal
- removed REF** (x9): MountingHole_2mm, MountingHole:MountingHole_2mm
- moved C1 77.7 mm to (117.3, 92.5)
- moved R1 77.7 mm to (87.3, 75.0)
- moved R2 77.7 mm to (107.3, 75.0)
- moved R3 77.7 mm to (127.3, 75.0)
- moved U1 77.7 mm to (107.8, 93.1)
- moved A1 77.7 mm to (130.8, 95.1)
- moved BT1 77.7 mm to (87.5, 60.0)
- moved C2 77.7 mm to (154.8, 65.0)
- moved J3 77.7 mm to (169.8, 72.5)
- moved J4 77.7 mm to (169.8, 67.5)
- moved R4 77.7 mm to (147.3, 75.0)
- moved R5 77.7 mm to (167.3, 75.0)
- moved SW1 77.7 mm to (169.8, 60.0)
- moved U2 77.7 mm to (142.3, 65.0)
Routing:
- net Net-(D1-Pad2): track 92.6 -> 0.00 mm
- net Net-(D1-Pad1): track 90.6 -> 0.00 mm
- net Net-(J1-Pad1): track 12.4 -> 0.00 mm
Other:
- board size 202.5 x 50 mm -> 100 x 50 mm
