File: hotdog-hw/hotdog-pcb/hotdog-pcb-front.kicad_sch (KiCad schematic)
At the start: 20 parts, among them J1 Conn_01x01, J2 Conn_01x01, J3 Conn_01x01, J4 Conn_01x01, SW1 SW_SPST, U1 NRF24L01_Breakout, U2 ME2108A

Commit message: Learned my lesson about PCB pooling
Parts:
- removed D1, D2, D3: LED, LED_THT:LED_D5.0mm, symbol Device:LED
- removed J1, J2: Conn_01x01, Connector_Wire:SolderWire-0.1sqmm_1x01_D0.4mm_OD1mm, symbol Connector_Generic:Conn_01x01
- removed R6: R, Resistor_THT:R_Axial_DIN0204_L3.6mm_D1.6mm_P5.08mm_Horizontal, symbol Device:R
- SW1: footprint (none) -> Button_Switch_THT:SW_CuK_OS102011MA1QN1_SPDT_Angled
Changed lines of the file:
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@@
   (junction (at 120.65 35.56) (diameter 0) (color 0 0 0 0)
   )
-  (junction (at 137.16 139.7) (diameter 0) (color 0 0 0 0)
-  )
   (junction (at 49.53 66.04) (diameter 0) (color 0 0 0 0)
   )
-  (junction (at 111.76 127) (diameter 0) (color 0 0 0 0)
-  )
   (junction (at 86.36 96.52) (diameter 0) (color 0 0 0 0)
   )
-  (junction (at 137.16 127) (diameter 0) (color 0 0 0 0)
-  )
   (junction (at 105.41 25.4) (diameter 0) (color 0 0 0 0)
   )
@@
   (junction (at 111.76 96.52) (diameter 0) (color 0 0 0 0)
   )
-  (junction (at 111.76 139.7) (diameter 0) (color 0 0 0 0)
-  )
   (junction (at 105.41 35.56) (diameter 0) (color 0 0 0 0)
   )
@@
     (stroke (width 0) (type default) (color 0 0 0 0))
   )
-  (wire (pts (xy 111.76 127) (xy 111.76 129.54))
-    (stroke (width 0) (type default) (color 0 0 0 0))
-  )
   (wire (pts (xy 149.86 63.5) (xy 96.52 63.5))
     (stroke (width 0) (type default) (color 0 0 0 0))
@@
     (stroke (width 0) (type default) (color 0 0 0 0))
   )
-  (wire (pts (xy 137.16 139.7) (xy 162.56 139.7))
-    (stroke (width 0) (type default) (color 0 0 0 0))
-  )
   (wire (pts (xy 86.36 30.48) (xy 49.53 30.48))
     (stroke (width 0) (type default) (color 0 0 0 0))
@@
     (stroke (width 0) (type default) (color 0 0 0 0))
   )
-  (wire (pts (xy 111.76 137.16) (xy 111.76 139.7))
-    (stroke (width 0) (type default) (color 0 0 0 0))
-  )
   (wire (pts (xy 62.23 78.74) (xy 71.12 78.74))
     (stroke (width 0) (type default) (color 0 0 0 0))
@@
     (stroke (width 0) (type default) (color 0 0 0 0))
   )
-  (wire (pts (xy 137.16 127) (xy 162.56 127))
-    (stroke (width 0) (type default) (color 0 0 0 0))
-  )
   (wire (pts (xy 83.82 86.36) (xy 83.82 96.52))
     (stroke (width 0) (type default) (color 0 0 0 0))
@@
     (stroke (width 0) (type default) (color 0 0 0 0))
   )
-  (wire (pts (xy 137.16 127) (xy 137.16 129.54))
-    (stroke (width 0) (type default) (color 0 0 0 0))
-  )
   (wire (pts (xy 128.27 25.4) (xy 139.7 25.4))
     (stroke (width 0) (type default) (color 0 0 0 0))
@@
     (stroke (width 0) (type default) (color 0 0 0 0))
   )
-  (wire (pts (xy 101.6 127) (xy 111.76 127))
-    (stroke (width 0) (type default) (color 0 0 0 0))
-  )
   (wire (pts (xy 68.58 71.12) (xy 71.12 71.12))
     (stroke (width 0) (type default) (color 0 0 0 0))
   )
-  (wire (pts (xy 162.56 139.7) (xy 162.56 137.16))
-    (stroke (width 0) (type default) (color 0 0 0 0))
-  )
   (wire (pts (xy 124.46 88.9) (xy 124.46 68.58))
     (stroke (width 0) (type default) (color 0 0 0 0))
@@
     (stroke (width 0) (type default) (color 0 0 0 0))
   )
-  (wire (pts (xy 86.36 139.7) (xy 111.76 139.7))
-    (stroke (width 0) (type default) (color 0 0 0 0))
-  )
-  (wire (pts (xy 111.76 139.7) (xy 137.16 139.7))
-    (stroke (width 0) (type default) (color 0 0 0 0))
-  )
-  (wire (pts (xy 111.76 127) (xy 137.16 127))
-    (stroke (width 0) (type default) (color 0 0 0 0))
-  )
   (wire (pts (xy 30.48 66.04) (xy 49.53 66.04))
     (stroke (width 0) (type default) (color 0 0 0 0))
   )
-  (wire (pts (xy 137.16 137.16) (xy 137.16 139.7))
-    (stroke (width 0) (type default) (color 0 0 0 0))
-  )
   (wire (pts (xy 137.16 66.04) (xy 96.52 66.04))
     (stroke (width 0) (type default) (color 0 0 0 0))
@@
     (stroke (width 0) (type default) (color 0 0 0 0))
   )
-  (wire (pts (xy 162.56 127) (xy 162.56 129.54))
-    (stroke (width 0) (type default) (color 0 0 0 0))
-  )
   (wire (pts (xy 62.23 73.66) (xy 71.12 73.66))
-    (stroke (width 0) (type default) (color 0 0 0 0))
-  )
-  (wire (pts (xy 86.36 127) (xy 93.98 127))
     (stroke (width 0) (type default) (color 0 0 0 0))
   )
@@
     (property "Reference" "SW1" (id 0) (at 129.54 30.48 0))
     (property "Value" "SW_SPST" (id 1) (at 129.54 33.02 0))
-    (property "Footprint" "" (id 2) (at 129.54 35.56 0)
+    (property "Footprint" "Button_Switch_THT:SW_CuK_OS102011MA1QN1_SPDT_Angled" (id 2) (at 129.54 35.56 0)
       (effects (font (size 1.27 1.27)) hide)
     )
     (property "Datasheet" "~" (id 3) (at 129.54 35.56 0)
-      (effects (font (size 1.27 1.27)) hide)
-    )
-    (pin "1")
-    (pin "2")
-  )
-  (symbol (lib_id "Device:LED") (at 111.76 133.35 90) (unit 1)
-    (in_bom yes) (on_board yes) (fields_autoplaced)
-    (property "Reference" "D1" (id 0) (at 115.57 133.6674 90)
-      (effects (font (size 1.27 1.27)) (justify right))
-    )
-    (property "Value" "LED" (id 1) (at 115.57 136.2074 90)
-      (effects (font (size 1.27 1.27)) (justify right))
-    )
-    (property "Footprint" "LED_THT:LED_D5.0mm" (id 2) (at 111.76 133.35 0)
-      (effects (font (size 1.27 1.27)) hide)
-    )
-    (property "Datasheet" "~" (id 3) (at 111.76 133.35 0)
-      (effects (font (size 1.27 1.27)) hide)
-    )
-    (pin "1")
-    (pin "2")
-  )
-  (symbol (lib_id "Device:LED") (at 137.16 133.35 90) (unit 1)
-    (in_bom yes) (on_board yes) (fields_autoplaced)
-    (property "Reference" "D2" (id 0) (at 140.97 133.6674 90)
-      (effects (font (size 1.27 1.27)) (justify right))
-    )
-    (property "Value" "LED" (id 1) (at 140.97 136.2074 90)
-      (effects (font (size 1.27 1.27)) (justify right))
-    )
-    (property "Footprint" "LED_THT:LED_D5.0mm" (id 2) (at 137.16 133.35 0)
-      (effects (font (size 1.27 1.27)) hide)
-    )
-    (property "Datasheet" "~" (id 3) (at 137.16 133.35 0)
       (effects (font (size 1.27 1.27)) hide)
     )
@@
     (pin "2")
   )
-  (symbol (lib_id "Connector_Generic:Conn_01x01") (at 81.28 139.7 180) (unit 1)
-    (in_bom yes) (on_board yes) (fields_autoplaced)
-    (property "Reference" "J2" (id 0) (at 81.28 133.35 0))
-    (property "Value" "Conn_01x01" (id 1) (at 81.28 135.89 0))
-    (property "Footprint" "Connector_Wire:SolderWire-0.1sqmm_1x01_D0.4mm_OD1mm" (id 2) (at 81.28 139.7 0)
-      (effects (font (size 1.27 1.27)) hide)
-    )
-    (property "Datasheet" "~" (id 3) (at 81.28 139.7 0)
-      (effects (font (size 1.27 1.27)) hide)
-    )
-    (pin "1")
-  )
   (symbol (lib_id "Sensor_Optical:LDR07") (at 111.76 92.71 0) (unit 1)
     (in_bom yes) (on_board yes) (fields_autoplaced)
@@
     (pin "1")
     (pin "2")
-  )
-  (symbol (lib_id "Connector_Generic:Conn_01x01") (at 81.28 127 180) (unit 1)
-    (in_bom yes) (on_board yes) (fields_autoplaced)
-    (property "Reference" "J1" (id 0) (at 81.28 120.65 0))
-    (property "Value" "Conn_01x01" (id 1) (at 81.28 123.19 0))
-    (property "Footprint" "Connector_Wire:SolderWire-0.1sqmm_1x01_D0.4mm_OD1mm" (id 2) (at 81.28 127 0)
-      (effects (font (size 1.27 1.27)) hide)
-    )
-    (property "Datasheet" "~" (id 3) (at 81.28 127 0)
-      (effects (font (size 1.27 1.27)) hide)
-    )
-    (pin "1")
   )
   (symbol (lib_id "Sensor_Optical:LDR07") (at 124.46 92.71 0) (unit 1)
@@
     )
     (pin "1")
-  )
-  (symbol (lib_id "Device:R") (at 97.79 127 270) (unit 1)
-    (in_bom yes) (on_board yes) (fields_autoplaced)
-    (property "Reference" "R6" (id 0) (at 97.79 120.65 90))
-    (property "Value" "R" (id 1) (at 97.79 123.19 90))
-    (property "Footprint" "Resistor_THT:R_Axial_DIN0204_L3.6mm_D1.6mm_P5.08mm_Horizontal" (id 2) (at 97.79 125.222 90)
-      (effects (font (size 1.27 1.27)) hide)
-    )
-    (property "Datasheet" "~" (id 3) (at 97.79 127 0)
-      (effects (font (size 1.27 1.27)) hide)
-    )
-    (pin "1")
-    (pin "2")
   )
   (symbol (lib_id "Regulator_Switching:R-78C5.0-1.0") (at 120.65 25.4 0) (mirror y) (unit 1)
@@
     (pin "3")
   )
-  (symbol (lib_id "Device:LED") (at 162.56 133.35 90) (unit 1)
-    (in_bom yes) (on_board yes) (fields_autoplaced)
-    (property "Reference" "D3" (id 0) (at 166.37 133.6674 90)
-      (effects (font (size 1.27 1.27)) (justify right))
-    )
-    (property "Value" "LED" (id 1) (at 166.37 136.2074 90)
-      (effects (font (size 1.27 1.27)) (justify right))
-    )
-    (property "Footprint" "LED_THT:LED_D5.0mm" (id 2) (at 162.56 133.35 0)
-      (effects (font (size 1.27 1.27)) hide)
-    )
-    (property "Datasheet" "~" (id 3) (at 162.56 133.35 0)
-      (effects (font (size 1.27 1.27)) hide)
-    )
-    (pin "1")
-    (pin "2")
-  )
   (sheet_instances
     (path "/" (page "1"))
@@
       (reference "C2") (unit 1) (value "C_Polarized") (footprint "Capacitor_THT:CP_Radial_D6.3mm_P2.50mm")
     )
-    (path "/2eabb083-b6e2-4c2c-a042-fcc3e5220a95"
-      (reference "D1") (unit 1) (value "LED") (footprint "LED_THT:LED_D5.0mm")
-    )
-    (path "/3c9cbf0a-9c83-436d-b6b9-ecf8d3017cbe"
-      (reference "D2") (unit 1) (value "LED") (footprint "LED_THT:LED_D5.0mm")
-    )
-    (path "/f6d5e9da-12e8-4206-8278-99c8e9695d12"
-      (reference "D3") (unit 1) (value "LED") (footprint "LED_THT:LED_D5.0mm")
-    )
-    (path "/9c8b39e2-a8ff-42cf-a3bc-36f609d4448b"
-      (reference "J1") (unit 1) (value "Conn_01x01") (footprint "Connector_Wire:SolderWire-0.1sqmm_1x01_D0.4mm_OD1mm")
-    )
-    (path "/8000f3ac-96eb-484e-a308-6f06b0dd2baa"
-      (reference "J2") (unit 1) (value "Conn_01x01") (footprint "Connector_Wire:SolderWire-0.1sqmm_1x01_D0.4mm_OD1mm")
-    )
     (path "/c51e6c18-e7b4-479e-9aba-1bcac67c96b5"
       (reference "J3") (unit 1) (value "Conn_01x01") (footprint "Connector_Wire:SolderWire-0.1sqmm_1x01_D0.4mm_OD1mm")
@@
       (reference "R5") (unit 1) (value "LDR07") (footprint "OptoDevice:R_LDR_5.1x4.3mm_P3.4mm_Vertical")
     )
-    (path "/d53a2abe-9358-439e-b2da-923cdba0460a"
-      (reference "R6") (unit 1) (value "R") (footprint "Resistor_THT:R_Axial_DIN0204_L3.6mm_D1.6mm_P5.08mm_Horizontal")
-    )
     (path "/2d56065f-684a-4165-b0e1-ca322bbb3f18"
